File: Buck-Boost-Switch-Mode-Power-Supply-Module.brd (EAGLE design)
At the start: 30.5 x 17.8 mm, 14 parts, among them IC1 LTM8055, P1 PINHEADER-7P, P2 PINHEADER-7P

Commit message: Changed to 18V output configuration used in RoboCup2023
Parts:
- R3: value 36.5k -> 45.3k
- R5: value 11k -> 6.98k
Changed lines of the file:
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@@
 <drawing>
 <settings>
-<setting alwaysvectorfont="yes"/>
+<setting alwaysvectorfont="no"/>
 <setting verticaltext="up"/>
 </settings>
@@
 <attribute name="VALUE" x="5.985" y="4.985" size="1.27" layer="27"/>
 </element>
-<element name="R3" library="rcl" library_urn="urn:adsk.eagle:library:334" package="R0603" package3d_urn="urn:adsk.eagle:package:23555/3" value="36.5k" x="-8.5725" y="4.1275" smashed="yes" rot="R270">
+<element name="R3" library="rcl" library_urn="urn:adsk.eagle:library:334" package="R0603" package3d_urn="urn:adsk.eagle:package:23555/3" value="45.3k" x="-8.5725" y="4.1275" smashed="yes" rot="R270">
 <attribute name="NAME" x="-9.8425" y="4.1275" size="0.8" layer="25" rot="R270" align="center"/>
 <attribute name="POPULARITY" value="77" x="-8.5725" y="4.1275" size="1.778" layer="27" rot="R270" display="off"/>
@@
 <attribute name="VALUE" x="1.5875" y="5.08" size="1.27" layer="27"/>
 </element>
-<element name="R5" library="rcl" library_urn="urn:adsk.eagle:library:334" package="R0603" package3d_urn="urn:adsk.eagle:package:23555/3" value="11k" x="-2.2225" y="6.985" smashed="yes" rot="R180">
+<element name="R5" library="rcl" library_urn="urn:adsk.eagle:library:334" package="R0603" package3d_urn="urn:adsk.eagle:package:23555/3" value="6.98k" x="-2.2225" y="6.985" smashed="yes" rot="R180">
 <attribute name="NAME" x="-2.2225" y="8.255" size="0.8" layer="25" rot="R180" align="center"/>
 <attribute name="POPULARITY" value="77" x="-2.2225" y="6.985" size="1.778" layer="27" rot="R180" display="off"/>
